File: CableAdapterBoard.kicad_pcb (KiCad board)
At the start: 6 copper layers, 102.3 x 46.1 mm, 20 parts, among them J1 IPL1-104-01-L-D-K, J2 IPL1-105-01-L-D-K, J21 1888174-6, J3 IPL1-105-01-X-D-K, J31 1888174-6

Commit message: Changed orientation of 36 pin minisas connectors to be CORRECT. old version needed a flip due to always top-to-bottom crossover format of these cables. corrected some labeling.
Parts:
- J21: renamed from J31; footprint Connector:TE_1888174-6 -> Tiles:TE_1888174-6
- J31: renamed from J21; footprint Connector:TE_1888174-6 -> Tiles:TE_1888174-6
Connections:
- J21 pad A10: unconnected-(J31-PadA10) -> DGND
- J21 pad A11: unconnected-(J31-PadA11) -> DGND
- J21 pad A13: /ASIC_GR -> /SACI_CLK_P
- J21 pad A14: /ASIC_PULSE -> /SACI_CLK_N
- J21 pad A16: unconnected-(J31-PadA16) -> /ASIC_SR0_P
- J21 pad A17: unconnected-(J31-PadA17) -> /ASIC_SR0_N
- J21 pad A2: /ASIC_SACI_SEL -> /SACI_RESP_P
- J21 pad A3: unconnected-(J31-PadA3) -> /SACI_RESP_N
- J21 pad A5: /ASIC_SampClkEn_P -> /SACI_CMD_P
- J21 pad A6: /ASIC_SampClkEn_N -> /SACI_CMD_N
- J21 pad A8: unconnected-(J31-PadA8) -> DGND
- J21 pad A9: unconnected-(J31-PadA9) -> DGND
- J21 pad B10: unconnected-(J31-PadB10) -> DGND
- J21 pad B11: unconnected-(J31-PadB11) -> DGND
- J21 pad B13: /SACI_CLK_P -> /ASIC_GR
- J21 pad B14: /SACI_CLK_N -> /ASIC_PULSE
- J21 pad B16: /ASIC_SR0_P -> unconnected-(J21-PadB16)
- J21 pad B17: /ASIC_SR0_N -> unconnected-(J21-PadB17)
- J21 pad B2: /SACI_RESP_P -> /ASIC_SACI_SEL
- J21 pad B3: /SACI_RESP_N -> unconnected-(J21-PadB3)
- J21 pad B5: /SACI_CMD_P -> /ASIC_SampClkEn_P
- J21 pad B6: /SACI_CMD_N -> /ASIC_SampClkEn_N
- J21 pad B8: unconnected-(J31-PadB8) -> DGND
- J21 pad B9: unconnected-(J31-PadB9) -> DGND
- J31 pad A10: unconnected-(J21-PadA10) -> DGND
- J31 pad A11: unconnected-(J21-PadA11) -> DGND
- J31 pad A13: unconnected-(J21-PadA13) -> /WORD_CLK_0_P
- J31 pad A14: unconnected-(J21-PadA14) -> /WORD_CLK_0_N
- J31 pad A16: unconnected-(J21-PadA16) -> /RD_CLK_P
- J31 pad A17: unconnected-(J21-PadA17) -> /RD_CLK_N
- J31 pad A2: /DATA_OUT_1_P -> /DATA_OUT_0_P
- J31 pad A3: /DATA_OUT_1_N -> /DATA_OUT_0_N
- J31 pad A8: unconnected-(J21-PadA8) -> DGND
- J31 pad A9: unconnected-(J21-PadA9) -> DGND
- J31 pad B10: unconnected-(J21-PadB10) -> DGND
- J31 pad B11: unconnected-(J21-PadB11) -> DGND
- J31 pad B13: /WORD_CLK_0_P -> unconnected-(J31-PadB13)
- J31 pad B14: /WORD_CLK_0_N -> unconnected-(J31-PadB14)
- J31 pad B16: /RD_CLK_P -> unconnected-(J31-PadB16)
- J31 pad B17: /RD_CLK_N -> unconnected-(J31-PadB17)
- J31 pad B2: /DATA_OUT_0_P -> /DATA_OUT_1_P
- J31 pad B3: /DATA_OUT_0_N -> /DATA_OUT_1_N
- J31 pad B8: unconnected-(J21-PadB8) -> DGND
- J31 pad B9: unconnected-(J21-PadB9) -> DGND
Routing:
- net /WORD_CLK_0_P: track 47.2 -> 32.4 mm, vias 3 -> 1
- net /WORD_CLK_0_N: track 45.4 -> 32.2 mm, vias 3 -> 1
- net /ASIC_SACI_SEL: track 23.0 -> 32.6 mm
- net /SACI_CMD_P: track 34.1 -> 25.7 mm
- net /SACI_CMD_N: track 35.4 -> 27.2 mm
- net /SACI_CLK_P: track 31.8 -> 26.0 mm
- net /SACI_CLK_N: track 33.3 -> 27.5 mm
- net /ASIC_PULSE: track 31.3 -> 37.0 mm, vias 0 -> 1
- net /ASIC_GR: track 34.3 -> 39.2 mm, vias 0 -> 1
- net /SACI_RESP_P: track 38.0 -> 33.6 mm
- net /ASIC_SampClkEn_P: track 48.8 -> 53.0 mm
- net /SACI_RESP_N: track 36.4 -> 32.3 mm
- net /ASIC_SR0_P: track 40.1 -> 36.3 mm
- net /ASIC_SR0_N: track 42.2 -> 38.5 mm
- net /ASIC_SampClkEn_N: track 46.2 -> 50.0 mm
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
Commit message: SOme backups and gerbers
Other:
- board text added: "This PCB uses JLCPCB JLC061611-7628 (Standard), whose PCB calculator is indicating a trace/space of 6.73 / 11"
- board text removed: "Stackup uses PCBWay standard 6-layer 1.6mm total thickness stackup for 1 oz copper. Recommended 6 mil space for easee of manufacture, 100 ohm differential impedance results in 9/9/9 trace space trace for their 1/1oz standard 6-layer stack, with In1 referencing top and In2 referencing bottom"
